File: Hardware/SparkFun_IMU_Breakout_ICM-20948.sch (EAGLE design)
At the start: 37 parts, among them U1 TXB0108DQSR, U2 9DoF IMU, U3 1.8V/100mA

Commit message: Fixed I2C heasder order
Also adjusted silkcreen labels to reflect the new order
Connections:
- net !CS: now also U1.A1; no longer U1.A4
- net !CS!_VIN: now also J3.6, U1.B1; no longer J3.3, U1.B4
- net AD0/SDO: now also U1.A2; no longer U1.A1
- net AD0/SDO_VIN: now also J3.5, U1.B2; no longer J3.6, U1.B1
- net SDA/SDI: now also U1.A4; no longer U1.A2
- net SDA/SDI_VIN: now also J3.3, U1.B4; no longer J3.5, U1.B2
Other:
- moved on the sheet: R2
Changed lines of the file:
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@@
 <attribute name="VALUE" x="33.02" y="112.014" size="1.778" layer="96" align="bottom-center"/>
 </instance>
-<instance part="SUPPLY4" gate="G$1" x="63.5" y="111.76">
-<attribute name="VALUE" x="63.5" y="114.554" size="1.778" layer="96" align="bottom-center"/>
+<instance part="SUPPLY4" gate="G$1" x="63.5" y="119.38">
+<attribute name="VALUE" x="63.5" y="122.174" size="1.778" layer="96" align="bottom-center"/>
 </instance>
 <instance part="GND6" gate="1" x="63.5" y="73.66">
@@
 <instance part="H2" gate="G$1" x="238.76" y="30.48"/>
 <instance part="H4" gate="G$1" x="241.3" y="30.48"/>
-<instance part="R2" gate="G$1" x="83.82" y="104.14" rot="R90">
-<attribute name="NAME" x="82.296" y="104.14" size="1.778" layer="95" font="vector" rot="R90" align="bottom-center"/>
-<attribute name="VALUE" x="85.344" y="104.14" size="1.778" layer="96" font="vector" rot="R90" align="top-center"/>
-</instance>
-<instance part="SUPPLY6" gate="G$1" x="83.82" y="111.76">
-<attribute name="VALUE" x="83.82" y="114.554" size="1.778" layer="96" align="bottom-center"/>
+<instance part="R2" gate="G$1" x="68.58" y="111.76" rot="R90">
+<attribute name="NAME" x="67.056" y="111.76" size="1.778" layer="95" font="vector" rot="R90" align="bottom-center"/>
+<attribute name="VALUE" x="70.104" y="111.76" size="1.778" layer="96" font="vector" rot="R90" align="top-center"/>
+</instance>
+<instance part="SUPPLY6" gate="G$1" x="68.58" y="119.38">
+<attribute name="VALUE" x="68.58" y="122.174" size="1.778" layer="96" align="bottom-center"/>
 </instance>
 <instance part="J2" gate="G$1" x="25.4" y="12.7">
@@
 </segment>
 <segment>
+<wire x1="30.48" y1="101.6" x2="35.56" y2="101.6" width="0.1524" layer="91"/>
+<label x="30.48" y="101.6" size="1.27" layer="95" rot="R180" xref="yes"/>
+<pinref part="U1" gate="G$1" pin="A2"/>
+</segment>
+</net>
+<net name="SDA/SDI" class="0">
+<segment>
+<pinref part="U2" gate="G$1" pin="SDA/SDI"/>
+<wire x1="83.82" y1="154.94" x2="81.28" y2="154.94" width="0.1524" layer="91"/>
+<label x="83.82" y="154.94" size="1.27" layer="95" xref="yes"/>
+</segment>
+<segment>
+<wire x1="30.48" y1="96.52" x2="35.56" y2="96.52" width="0.1524" layer="91"/>
+<label x="30.48" y="96.52" size="1.27" layer="95" rot="R180" xref="yes"/>
+<pinref part="U1" gate="G$1" pin="A4"/>
+</segment>
+</net>
+<net name="SCL/SCLK" class="0">
+<segment>
+<pinref part="U2" gate="G$1" pin="SCL/SCLK"/>
+<wire x1="83.82" y1="157.48" x2="81.28" y2="157.48" width="0.1524" layer="91"/>
+<label x="83.82" y="157.48" size="1.27" layer="95" xref="yes"/>
+</segment>
+<segment>
+<wire x1="30.48" y1="99.06" x2="35.56" y2="99.06" width="0.1524" layer="91"/>
+<label x="30.48" y="99.06" size="1.27" layer="95" rot="R180" xref="yes"/>
+<pinref part="U1" gate="G$1" pin="A3"/>
+</segment>
+</net>
+<net name="!CS" class="0">
+<segment>
+<pinref part="U2" gate="G$1" pin="!CS"/>
+<label x="83.82" y="160.02" size="1.27" layer="95" xref="yes"/>
+<wire x1="83.82" y1="160.02" x2="81.28" y2="160.02" width="0.1524" layer="91"/>
+</segment>
+<segment>
 <wire x1="30.48" y1="104.14" x2="35.56" y2="104.14" width="0.1524" layer="91"/>
 <label x="30.48" y="104.14" size="1.27" layer="95" rot="R180" xref="yes"/>
 <pinref part="U1" gate="G$1" pin="A1"/>
-</segment>
-</net>
-<net name="SDA/SDI" class="0">
-<segment>
-<pinref part="U2" gate="G$1" pin="SDA/SDI"/>
-<wire x1="83.82" y1="154.94" x2="81.28" y2="154.94" width="0.1524" layer="91"/>
-<label x="83.82" y="154.94" size="1.27" layer="95" xref="yes"/>
-</segment>
-<segment>
-<wire x1="30.48" y1="101.6" x2="35.56" y2="101.6" width="0.1524" layer="91"/>
-<label x="30.48" y="101.6" size="1.27" layer="95" rot="R180" xref="yes"/>
-<pinref part="U1" gate="G$1" pin="A2"/>
-</segment>
-</net>
-<net name="SCL/SCLK" class="0">
-<segment>
-<pinref part="U2" gate="G$1" pin="SCL/SCLK"/>
-<wire x1="83.82" y1="157.48" x2="81.28" y2="157.48" width="0.1524" layer="91"/>
-<label x="83.82" y="157.48" size="1.27" layer="95" xref="yes"/>
-</segment>
-<segment>
-<wire x1="30.48" y1="99.06" x2="35.56" y2="99.06" width="0.1524" layer="91"/>
-<label x="30.48" y="99.06" size="1.27" layer="95" rot="R180" xref="yes"/>
-<pinref part="U1" gate="G$1" pin="A3"/>
-</segment>
-</net>
-<net name="!CS" class="0">
-<segment>
-<pinref part="U2" gate="G$1" pin="!CS"/>
-<label x="83.82" y="160.02" size="1.27" layer="95" xref="yes"/>
-<wire x1="83.82" y1="160.02" x2="81.28" y2="160.02" width="0.1524" layer="91"/>
-</segment>
-<segment>
-<wire x1="30.48" y1="96.52" x2="35.56" y2="96.52" width="0.1524" layer="91"/>
-<label x="30.48" y="96.52" size="1.27" layer="95" rot="R180" xref="yes"/>
-<pinref part="U1" gate="G$1" pin="A4"/>
 </segment>
 </net>
@@
 <segment>
 <pinref part="U1" gate="G$1" pin="VCCB"/>
-<wire x1="63.5" y1="111.76" x2="63.5" y2="93.98" width="0.1524" layer="91"/>
+<wire x1="63.5" y1="119.38" x2="63.5" y2="93.98" width="0.1524" layer="91"/>
 <wire x1="63.5" y1="93.98" x2="60.96" y2="93.98" width="0.1524" layer="91"/>
 <pinref part="SUPPLY4" gate="G$1" pin="VIN"/>
@@
 <pinref part="SUPPLY6" gate="G$1" pin="VIN"/>
 <pinref part="R2" gate="G$1" pin="2"/>
-<wire x1="83.82" y1="111.76" x2="83.82" y2="109.22" width="0.1524" layer="91"/>
+<wire x1="68.58" y1="119.38" x2="68.58" y2="116.84" width="0.1524" layer="91"/>
 </segment>
 <segment>
@@
 <net name="AD0/SDO_VIN" class="0">
 <segment>
-<wire x1="66.04" y1="104.14" x2="60.96" y2="104.14" width="0.1524" layer="91"/>
-<label x="66.04" y="104.14" size="1.27" layer="95" xref="yes"/>
-<pinref part="U1" gate="G$1" pin="B1"/>
-</segment>
-<segment>
-<pinref part="J3" gate="G$1" pin="6"/>
-<wire x1="81.28" y1="22.86" x2="76.2" y2="22.86" width="0.1524" layer="91"/>
-<label x="81.28" y="22.86" size="1.27" layer="95" xref="yes"/>
+<wire x1="66.04" y1="101.6" x2="60.96" y2="101.6" width="0.1524" layer="91"/>
+<label x="66.04" y="101.6" size="1.27" layer="95" xref="yes"/>
+<pinref part="U1" gate="G$1" pin="B2"/>
+</segment>
+<segment>
+<wire x1="81.28" y1="20.32" x2="76.2" y2="20.32" width="0.1524" layer="91"/>
+<label x="81.28" y="20.32" size="1.27" layer="95" xref="yes"/>
+<pinref part="J3" gate="G$1" pin="5"/>
 </segment>
 <segment>
@@
 <net name="SDA/SDI_VIN" class="0">
 <segment>
-<wire x1="66.04" y1="101.6" x2="60.96" y2="101.6" width="0.1524" layer="91"/>
-<label x="66.04" y="101.6" size="1.27" layer="95" xref="yes"/>
-<pinref part="U1" gate="G$1" pin="B2"/>
+<wire x1="66.04" y1="96.52" x2="60.96" y2="96.52" width="0.1524" layer="91"/>
+<label x="66.04" y="96.52" size="1.27" layer="95" xref="yes"/>
+<pinref part="U1" gate="G$1" pin="B4"/>
 </segment>
 <segment>
@@
 </segment>
 <segment>
-<pinref part="J3" gate="G$1" pin="5"/>
-<wire x1="81.28" y1="20.32" x2="76.2" y2="20.32" width="0.1524" layer="91"/>
-<label x="81.28" y="20.32" size="1.27" layer="95" xref="yes"/>
+<wire x1="81.28" y1="15.24" x2="76.2" y2="15.24" width="0.1524" layer="91"/>
+<label x="81.28" y="15.24" size="1.27" layer="95" xref="yes"/>
+<pinref part="J3" gate="G$1" pin="3"/>
 </segment>
 <segment>
@@
 <net name="!CS!_VIN" class="0">
 <segment>
-<wire x1="86.36" y1="96.52" x2="83.82" y2="96.52" width="0.1524" layer="91"/>
-<label x="86.36" y="96.52" size="1.27" layer="95" xref="yes"/>
+<wire x1="71.12" y1="104.14" x2="68.58" y2="104.14" width="0.1524" layer="91"/>
+<label x="71.12" y="104.14" size="1.27" layer="95" xref="yes"/>
 <pinref part="R2" gate="G$1" pin="1"/>
-<wire x1="83.82" y1="99.06" x2="83.82" y2="96.52" width="0.1524" layer="91"/>
-<pinref part="U1" gate="G$1" pin="B4"/>
-<wire x1="60.96" y1="96.52" x2="83.82" y2="96.52" width="0.1524" layer="91"/>
-<junction x="83.82" y="96.52"/>
-</segment>
-<segment>
-<pinref part="J3" gate="G$1" pin="3"/>
-<wire x1="81.28" y1="15.24" x2="76.2" y2="15.24" width="0.1524" layer="91"/>
-<label x="81.28" y="15.24" size="1.27" layer="95" xref="yes"/>
-</segment>
-</net>
+<wire x1="68.58" y1="106.68" x2="68.58" y2="104.14" width="0.1524" layer="91"/>
+<wire x1="60.96" y1="104.14" x2="68.58" y2="104.14" width="0.1524" layer="91"/>
+<junction x="68.58" y="104.14"/>
+<pinref part="U1" gate="G$1" pin="B1"/>
+</segment>
+<segment>
+<wire x1="81.28" y1="22.86" x2="76.2" y2="22.86" width="0.1524" layer="91"/>
+<label x="81.28" y="22.86" size="1.27" layer="95" xref="yes"/>
+<pinref part="J3" gate="G$1" pin="6"/>
+</segment>
+</net>

Commit message: Swap TXB0108 for TXS0108 - still needs last check, design review, and finalization
Parts:
- U1: value TXB0108DQSR -> -VFQFN_20; device SparkFun-IC-Comms:TXB0108 -> SparkFun-IC-Comms:TXS0108-VFQFN_20
Connections:
- net GND: no longer J4.6
- net VIN: now also J4.6
Changed lines of the file:
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@@
 <part name="SUPPLY1" library="SparkFun-PowerSymbols" deviceset="1.8V" device=""/>
 <part name="U3" library="SparkFun-IC-Power" deviceset="V_REG_SP6214" device="-1.8V" value="1.8V/100mA"/>
-<part name="U1" library="SparkFun-IC-Comms" deviceset="TXB0108" device="" value="TXB0108DQSR"/>
 <part name="SUPPLY8" library="SparkFun-PowerSymbols" deviceset="VIN" device=""/>
 <part name="C4" library="SparkFun-Capacitors" deviceset="1.0UF" device="-0603-16V-10%-X7R" value="1.0uF"/>
@@
 <part name="JP2" library="SparkFun-Jumpers" deviceset="JUMPER-SMT_2_NO" device="_SILK" value="AD0"/>
 <part name="GND11" library="SparkFun-PowerSymbols" deviceset="GND" device=""/>
+<part name="U1" library="SparkFun-IC-Comms" deviceset="TXS0108" device="-VFQFN_20" value="-VFQFN_20"/>
+<part name="SUPPLY13" library="SparkFun-PowerSymbols" deviceset="VIN" device=""/>
 </parts>
 <sheets>
@@
 <attribute name="VALUE" x="180.34" y="81.026" size="1.778" layer="96" font="vector" align="top-left"/>
 </instance>
-<instance part="U1" gate="G$1" x="48.26" y="93.98">
-<attribute name="VALUE" x="38.1" y="77.47" size="1.778" layer="96" align="center-left"/>
-<attribute name="NAME" x="38.1" y="107.95" size="1.778" layer="95" align="center-left"/>
-</instance>
 <instance part="SUPPLY8" gate="G$1" x="165.1" y="96.52">
 <attribute name="VALUE" x="165.1" y="99.314" size="1.778" layer="96" align="bottom-center"/>
@@
 <attribute name="VALUE" x="137.16" y="134.366" size="1.778" layer="96" align="top-center"/>
 </instance>
+<instance part="U1" gate="G$1" x="48.26" y="93.98"/>
+<instance part="SUPPLY13" gate="G$1" x="116.84" y="25.4">
+<attribute name="VALUE" x="116.84" y="28.194" size="1.778" layer="96" align="bottom-center"/>
+</instance>
 </instances>
 <busses>
@@
 </segment>
 <segment>
-<pinref part="U1" gate="G$1" pin="GND"/>
 <wire x1="60.96" y1="91.44" x2="63.5" y2="91.44" width="0.1524" layer="91"/>
 <wire x1="63.5" y1="91.44" x2="63.5" y2="76.2" width="0.1524" layer="91"/>
 <pinref part="GND6" gate="1" pin="GND"/>
+<pinref part="U1" gate="G$1" pin="GND"/>
 </segment>
 <segment>
@@
 </segment>
 <segment>
-<pinref part="J4" gate="G$1" pin="6"/>
-<wire x1="114.3" y1="22.86" x2="116.84" y2="22.86" width="0.1524" layer="91"/>
-<wire x1="116.84" y1="22.86" x2="116.84" y2="10.16" width="0.1524" layer="91"/>
 <pinref part="J4" gate="G$1" pin="1"/>
 <wire x1="116.84" y1="10.16" x2="116.84" y2="7.62" width="0.1524" layer="91"/>
 <wire x1="114.3" y1="10.16" x2="116.84" y2="10.16" width="0.1524" layer="91"/>
-<junction x="116.84" y="10.16"/>
 <pinref part="GND10" gate="1" pin="GND"/>
 </segment>
@@
 </segment>
 <segment>
-<pinref part="U1" gate="G$1" pin="A8"/>
 <wire x1="30.48" y1="81.28" x2="35.56" y2="81.28" width="0.1524" layer="91"/>
 <label x="30.48" y="81.28" size="1.27" layer="95" rot="R180" xref="yes"/>
+<pinref part="U1" gate="G$1" pin="A8"/>
 </segment>
 </net>
@@
 </segment>
 <segment>
-<pinref part="U1" gate="G$1" pin="A7"/>
 <wire x1="30.48" y1="83.82" x2="35.56" y2="83.82" width="0.1524" layer="91"/>
 <label x="30.48" y="83.82" size="1.27" layer="95" rot="R180" xref="yes"/>
+<pinref part="U1" gate="G$1" pin="A7"/>
 </segment>
 </net>
@@
 </segment>
 <segment>
-<pinref part="U1" gate="G$1" pin="OE"/>
 <wire x1="35.56" y1="91.44" x2="33.02" y2="91.44" width="0.1524" layer="91"/>
 <wire x1="33.02" y1="91.44" x2="33.02" y2="93.98" width="0.1524" layer="91"/>
-<pinref part="U1" gate="G$1" pin="VCCA"/>
 <wire x1="33.02" y1="93.98" x2="35.56" y2="93.98" width="0.1524" layer="91"/>
 <wire x1="33.02" y1="93.98" x2="33.02" y2="109.22" width="0.1524" layer="91"/>
 <junction x="33.02" y="93.98"/>
 <pinref part="SUPPLY2" gate="G$1" pin="1.8V"/>
+<pinref part="U1" gate="G$1" pin="VCCA"/>
+<pinref part="U1" gate="G$1" pin="OE"/>
 </segment>
 <segment>
@@
 </segment>
 <segment>
-<pinref part="U1" gate="G$1" pin="VCCB"/>
 <wire x1="63.5" y1="119.38" x2="63.5" y2="93.98" width="0.1524" layer="91"/>
 <wire x1="63.5" y1="93.98" x2="60.96" y2="93.98" width="0.1524" layer="91"/>
 <pinref part="SUPPLY4" gate="G$1" pin="VIN"/>
+<pinref part="U1" gate="G$1" pin="VCCB"/>
 </segment>
 <segment>
@@
 <wire x1="137.16" y1="167.64" x2="137.16" y2="165.1" width="0.1524" layer="91"/>
 </segment>
+<segment>
+<pinref part="J4" gate="G$1" pin="6"/>
+<wire x1="114.3" y1="22.86" x2="116.84" y2="22.86" width="0.1524" layer="91"/>
+<pinref part="SUPPLY13" gate="G$1" pin="VIN"/>
+<wire x1="116.84" y1="25.4" x2="116.84" y2="22.86" width="0.1524" layer="91"/>
+</segment>
 </net>
 <net name="AUX_CL_VIN" class="0">
@@
 <segment>
 <label x="66.04" y="99.06" size="1.27" layer="95" xref="yes"/>
+<wire x1="60.96" y1="99.06" x2="66.04" y2="99.06" width="0.1524" layer="91"/>
 <pinref part="U1" gate="G$1" pin="B3"/>
-<wire x1="60.96" y1="99.06" x2="66.04" y2="99.06" width="0.1524" layer="91"/>
 </segment>
 <segment>
@@
 <net name="FSYNC_VIN" class="0">
 <segment>
-<pinref part="U1" gate="G$1" pin="B7"/>
 <wire x1="88.9" y1="83.82" x2="78.74" y2="83.82" width="0.1524" layer="91"/>
 <label x="88.9" y="83.82" size="1.27" layer="95" xref="yes"/>
@@
 <wire x1="78.74" y1="76.2" x2="78.74" y2="83.82" width="0.1524" layer="91"/>
 <junction x="78.74" y="83.82"/>
+<pinref part="U1" gate="G$1" pin="B7"/>
 </segment>
 <segment>
@@
 <net name="INT_VIN" class="0">
 <segment>
-<pinref part="U1" gate="G$1" pin="B8"/>
 <wire x1="88.9" y1="81.28" x2="86.36" y2="81.28" width="0.1524" layer="91"/>
 <label x="88.9" y="81.28" size="1.27" layer="95" xref="yes"/>
@@
 <wire x1="86.36" y1="76.2" x2="86.36" y2="81.28" width="0.1524" layer="91"/>
 <junction x="86.36" y="81.28"/>
-</segment>
-<segment>
+<pinref part="U1" gate="G$1" pin="B8"/>
+</segment>
+<segment>
