File: Hardware/FetEvaluation/SparkFun_IMU_Breakout_ICM-20948_FET_EVAL.sch (EAGLE design)
At the start: 60 parts, among them Q1 DMN2005LP4K-7, Q10 RE1C002UN, Q11 DMN2005LP4K-7, Q12 RE1C002UN, Q13 DMN2005LP4K-7, Q14 RE1C002UN, Q15 DMN2005LP4K-7, Q16 RE1C002UN, Q2 RE1C002UN, Q3 DMN2005LP4K-7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

Commit message: Laid out board for MOSFET trick evaluation (prototype)
Parts:
- added U1, U10, U11, U12, U13, U14, U15, U16, U17, U18, U4, U5, U6, U7, U8, U9: TP, new_fets:TP
Connections:
- net !CS: now also U17.1
- net !CS!_VIN: now also U18.1
- net AD0/SDO: now also U15.1
- net AD0/SDO_VIN: now also U16.1
- net AUX_CL: now also U5.1
- net AUX_CL_VIN: now also J4.5, U6.1; no longer J4.3
- net AUX_DA: now also U1.1
- net AUX_DA_VIN: now also J4.4, U4.1; no longer J4.2
- net FSYNC: now also U8.1
- net FSYNC_VIN: now also J4.3, U7.1; no longer J4.4
- net INT: now also U9.1
- net INT_VIN: now also J4.2, U10.1; no longer J4.5
- net SCL/SCLK: now also U13.1
- net SCL/SCLK_VIN: now also U14.1
- net SDA/SDI: now also U11.1
- net SDA/SDI_VIN: now also U12.1
Changed lines of the file:
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@@
 <part name="SUPPLY29" library="SparkFun-PowerSymbols" deviceset="VIN" device=""/>
 <part name="SUPPLY2" library="SparkFun-PowerSymbols" deviceset="VIN" device=""/>
+<part name="U1" library="new_fets" deviceset="TP" device=""/>
+<part name="U4" library="new_fets" deviceset="TP" device=""/>
+<part name="U5" library="new_fets" deviceset="TP" device=""/>
+<part name="U6" library="new_fets" deviceset="TP" device=""/>
+<part name="U7" library="new_fets" deviceset="TP" device=""/>
+<part name="U8" library="new_fets" deviceset="TP" device=""/>
+<part name="U9" library="new_fets" deviceset="TP" device=""/>
+<part name="U10" library="new_fets" deviceset="TP" device=""/>
+<part name="U11" library="new_fets" deviceset="TP" device=""/>
+<part name="U12" library="new_fets" deviceset="TP" device=""/>
+<part name="U13" library="new_fets" deviceset="TP" device=""/>
+<part name="U14" library="new_fets" deviceset="TP" device=""/>
+<part name="U15" library="new_fets" deviceset="TP" device=""/>
+<part name="U16" library="new_fets" deviceset="TP" device=""/>
+<part name="U17" library="new_fets" deviceset="TP" device=""/>
+<part name="U18" library="new_fets" deviceset="TP" device=""/>
 </parts>
 <sheets>
@@
 <attribute name="VALUE" x="254" y="231.394" size="1.778" layer="96" align="bottom-center"/>
 </instance>
+<instance part="U1" gate="G$1" x="393.7" y="231.14" rot="R180"/>
+<instance part="U4" gate="G$1" x="416.56" y="231.14"/>
+<instance part="U5" gate="G$1" x="393.7" y="182.88" rot="R180"/>
+<instance part="U6" gate="G$1" x="416.56" y="182.88"/>
+<instance part="U7" gate="G$1" x="416.56" y="134.62"/>
+<instance part="U8" gate="G$1" x="393.7" y="134.62" rot="R180"/>
+<instance part="U9" gate="G$1" x="393.7" y="86.36" rot="R180"/>
+<instance part="U10" gate="G$1" x="416.56" y="86.36"/>
+<instance part="U11" gate="G$1" x="345.44" y="86.36" rot="R180"/>
+<instance part="U12" gate="G$1" x="368.3" y="86.36"/>
+<instance part="U13" gate="G$1" x="345.44" y="134.62" rot="R180"/>
+<instance part="U14" gate="G$1" x="368.3" y="134.62"/>
+<instance part="U15" gate="G$1" x="345.44" y="182.88" rot="R180"/>
+<instance part="U16" gate="G$1" x="368.3" y="182.88"/>
+<instance part="U17" gate="G$1" x="345.44" y="231.14" rot="R180"/>
+<instance part="U18" gate="G$1" x="368.3" y="231.14"/>
 </instances>
 <busses>
@@
 <junction x="393.7" y="96.52"/>
 <label x="391.16" y="96.52" size="1.27" layer="95" rot="R180" xref="yes"/>
+<pinref part="U9" gate="G$1" pin="1"/>
+<wire x1="393.7" y1="86.36" x2="396.24" y2="86.36" width="0.1524" layer="91" style="longdash"/>
+<junction x="396.24" y="86.36"/>
 </segment>
 </net>
@@
 <junction x="393.7" y="144.78"/>
 <label x="391.16" y="144.78" size="1.27" layer="95" rot="R180" xref="yes"/>
+<pinref part="U8" gate="G$1" pin="1"/>
+<wire x1="396.24" y1="134.62" x2="393.7" y2="134.62" width="0.1524" layer="91" style="longdash"/>
+<junction x="396.24" y="134.62"/>
 </segment>
 </net>
@@
 <junction x="345.44" y="193.04"/>
 <label x="342.9" y="193.04" size="1.27" layer="95" rot="R180" xref="yes"/>
+<pinref part="U15" gate="G$1" pin="1"/>
+<wire x1="345.44" y1="182.88" x2="347.98" y2="182.88" width="0.1524" layer="91" style="longdash"/>
+<junction x="347.98" y="182.88"/>
 </segment>
 </net>
@@
 <junction x="345.44" y="96.52"/>
 <label x="342.9" y="96.52" size="1.27" layer="95" rot="R180" xref="yes"/>
+<pinref part="U11" gate="G$1" pin="1"/>
+<wire x1="345.44" y1="86.36" x2="347.98" y2="86.36" width="0.1524" layer="91" style="longdash"/>
+<junction x="347.98" y="86.36"/>
 </segment>
 </net>
@@
 <junction x="345.44" y="144.78"/>
 <label x="342.9" y="144.78" size="1.27" layer="95" rot="R180" xref="yes"/>
+<pinref part="U13" gate="G$1" pin="1"/>
+<wire x1="345.44" y1="134.62" x2="347.98" y2="134.62" width="0.1524" layer="91" style="longdash"/>
+<junction x="347.98" y="134.62"/>
 </segment>
 </net>
@@
 <junction x="345.44" y="241.3"/>
 <label x="342.9" y="241.3" size="1.27" layer="95" rot="R180" xref="yes"/>
+<pinref part="U17" gate="G$1" pin="1"/>
+<wire x1="345.44" y1="231.14" x2="347.98" y2="231.14" width="0.1524" layer="91" style="longdash"/>
+<junction x="347.98" y="231.14"/>
 </segment>
 </net>
@@
 <junction x="393.7" y="241.3"/>
 <label x="391.16" y="241.3" size="1.27" layer="95" rot="R180" xref="yes"/>
+<pinref part="U1" gate="G$1" pin="1"/>
+<wire x1="393.7" y1="231.14" x2="396.24" y2="231.14" width="0.1524" layer="91" style="longdash"/>
+<junction x="396.24" y="231.14"/>
 </segment>
 </net>
@@
 <junction x="393.7" y="193.04"/>
 <label x="391.16" y="193.04" size="1.27" layer="95" rot="R180" xref="yes"/>
+<pinref part="U5" gate="G$1" pin="1"/>
+<wire x1="393.7" y1="182.88" x2="396.24" y2="182.88" width="0.1524" layer="91" style="longdash"/>
+<junction x="396.24" y="182.88"/>
 </segment>
 </net>
@@
 <net name="AUX_CL_VIN" class="0">
 <segment>
-<wire x1="121.92" y1="63.5" x2="116.84" y2="63.5" width="0.1524" layer="91"/>
-<label x="121.92" y="63.5" size="1.27" layer="95" font="vector" xref="yes"/>
-<pinref part="J4" gate="G$1" pin="3"/>
+<wire x1="119.38" y1="68.58" x2="116.84" y2="68.58" width="0.1524" layer="91"/>
+<label x="119.38" y="68.58" size="1.27" layer="95" font="vector" xref="yes"/>
+<pinref part="J4" gate="G$1" pin="5"/>
 </segment>
 <segment>
@@
 <junction x="414.02" y="193.04"/>
 <label x="416.56" y="193.04" size="1.27" layer="95" xref="yes"/>
+<pinref part="U6" gate="G$1" pin="1"/>
+<wire x1="414.02" y1="182.88" x2="416.56" y2="182.88" width="0.1524" layer="91" style="longdash"/>
+<junction x="414.02" y="182.88"/>
 </segment>
 </net>
 <net name="AUX_DA_VIN" class="0">
 <segment>
-<wire x1="121.92" y1="60.96" x2="116.84" y2="60.96" width="0.1524" layer="91"/>
-<label x="121.92" y="60.96" size="1.27" layer="95" font="vector" xref="yes"/>
-<pinref part="J4" gate="G$1" pin="2"/>
+<wire x1="119.38" y1="66.04" x2="116.84" y2="66.04" width="0.1524" layer="91"/>
+<label x="119.38" y="66.04" size="1.27" layer="95" font="vector" xref="yes"/>
+<pinref part="J4" gate="G$1" pin="4"/>
 </segment>
 <segment>
@@
 <wire x1="411.48" y1="243.84" x2="411.48" y2="241.3" width="0.1524" layer="91"/>
 <junction x="411.48" y="241.3"/>
+<pinref part="U4" gate="G$1" pin="1"/>
+<wire x1="416.56" y1="231.14" x2="414.02" y2="231.14" width="0.1524" layer="91" style="longdash"/>
+<junction x="414.02" y="231.14"/>
 </segment>
 </net>
@@
 <junction x="365.76" y="193.04"/>
 <label x="368.3" y="193.04" size="1.27" layer="95" xref="yes"/>
+<pinref part="U16" gate="G$1" pin="1"/>
+<wire x1="365.76" y1="182.88" x2="368.3" y2="182.88" width="0.1524" layer="91" style="longdash"/>
+<junction x="365.76" y="182.88"/>
 </segment>
 </net>
@@
 <junction x="365.76" y="96.52"/>
 <label x="368.3" y="96.52" size="1.27" layer="95" xref="yes"/>
+<pinref part="U12" gate="G$1" pin="1"/>
+<wire x1="365.76" y1="86.36" x2="368.3" y2="86.36" width="0.1524" layer="91" style="longdash"/>
+<junction x="365.76" y="86.36"/>
 </segment>
 </net>
@@
 <junction x="365.76" y="144.78"/>
 <label x="368.3" y="144.78" size="1.27" layer="95" xref="yes"/>
+<pinref part="U14" gate="G$1" pin="1"/>
+<wire x1="365.76" y1="134.62" x2="368.3" y2="134.62" width="0.1524" layer="91" style="longdash"/>
+<junction x="365.76" y="134.62"/>
 </segment>
 </net>
@@
 <junction x="365.76" y="241.3"/>
 <label x="368.3" y="241.3" size="1.27" layer="95" xref="yes"/>
+<pinref part="U18" gate="G$1" pin="1"/>
+<wire x1="368.3" y1="231.14" x2="365.76" y2="231.14" width="0.1524" layer="91" style="longdash"/>
+<junction x="365.76" y="231.14"/>
 </segment>
 </net>
 <net name="FSYNC_VIN" class="0">
 <segment>
-<wire x1="121.92" y1="66.04" x2="116.84" y2="66.04" width="0.1524" layer="91"/>
-<label x="121.92" y="66.04" size="1.27" layer="95" font="vector" xref="yes"/>
-<pinref part="J4" gate="G$1" pin="4"/>
+<wire x1="119.38" y1="63.5" x2="116.84" y2="63.5" width="0.1524" layer="91"/>
+<label x="119.38" y="63.5" size="1.27" layer="95" font="vector" xref="yes"/>
+<pinref part="J4" gate="G$1" pin="3"/>
 </segment>
 <segment>
@@
 <junction x="414.02" y="144.78"/>
 <label x="416.56" y="144.78" size="1.27" layer="95" xref="yes"/>
+<pinref part="U7" gate="G$1" pin="1"/>
+<wire x1="414.02" y1="134.62" x2="416.56" y2="134.62" width="0.1524" layer="91" style="longdash"/>
+<junction x="414.02" y="134.62"/>
 </segment>
 </net>
 <net name="INT_VIN" class="0">
 <segment>
-<wire x1="121.92" y1="68.58" x2="116.84" y2="68.58" width="0.1524" layer="91"/>
-<label x="121.92" y="68.58" size="1.27" layer="95" font="vector" xref="yes"/>
-<pinref part="J4" gate="G$1" pin="5"/>
+<wire x1="119.38" y1="60.96" x2="116.84" y2="60.96" width="0.1524" layer="91"/>
+<label x="119.38" y="60.96" size="1.27" layer="95" font="vector" xref="yes"/>
+<pinref part="J4" gate="G$1" pin="2"/>
 </segment>
 <segment>
@@
 <junction x="414.02" y="96.52"/>
 <label x="416.56" y="96.52" size="1.27" layer="95" xref="yes"/>
-</segment>
-</net>
+<pinref part="U10" gate="G$1" pin="1"/>
+<wire x1="414.02" y1="86.36" x2="416.56" y2="86.36" width="0.1524" layer="91" style="longdash"/>
+<junction x="414.02" y="86.36"/>
+</segment>
+</net>

Commit message: Changes from design review
Connections:
- net AUX_CL_VIN_JMP renamed N$4
- net AUX_DA_VIN_JMP renamed N$5
- net SCL/SCLK_VIN_JMP renamed N$2
- net SDA/SDI_VIN_JMP renamed N$3
Other:
- note added: "Address Option"
- note added: "I2C Level Shifting + Pullup Disconnects"
- note added: "SPI / Interrupt Level Shifting"
- note removed: "Level Shifting"
- note removed: "Options"
- moved on the sheet: C4, D1, JP2, JP3, JP4, JP5, Q1, Q10, Q11, Q12, Q13, Q14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
