File: Hardware/FetEvaluation/Production/SparkFun_IMU_Breakout_ICM-20948_FET_EVAL-Panel.brd (EAGLE design)
At the start: 31.8 x 25.4 mm, 118 parts, among them Q1 DMN2005LP4K-7, Q10 RE1C002UN, Q11 DMN2005LP4K-7, Q12 RE1C002UN, Q13 DMN2005LP4K-7, Q14 RE1C002UN, Q15 DMN2005LP4K-7, Q16 RE1C002UN, Q2 RE1C002UN, Q3 DMN2005LP4K-7, Q4 RE1C002UN, Q5 DMN2005LP4K-7, Q6 RE1C002UN, Q7 DMN2005LP4K-7, Q8 RE1C002UN, Q9 DMN2005LP4K-7, U1 TP, U10 TP, U11 TP, U12 TP, U13 TP, U14 TP, U15 TP, U16 TP, U17 TP, U18 TP, U2 9DoF IMU, U3 1.8V/100mA, U4 TP, U5 TP, U6 TP, U7 TP, U8 TP, U9 TP

Commit message: Changes from design review
Parts:
- removed FRAME2: FRAME-LEDGER, SparkFun-Aesthetics:CREATIVE_COMMONS
- added C10, C13, C14, C17, C18, C21, C22, C5, C6, C9: 0.1uF, SparkFun-Capacitors:0603
- added C11, C12, C15, C16, C19, C20, C23, C24, C7, C8: 1.0uF, SparkFun-Capacitors:0603
- added D2, D3, D4, D5, D6: RED, SparkFun-LED:LED-0603
- added E$1, E$2: (no value), SparkFun-Aesthetics:FIDUCIAL-1X2
- added E$3: (no value), SparkFun-Retired:FIDUCIAL-1.5X3
- added FD10, FD11, FD12, FD13, FD14, FD15, FD16, FD17, FD18, FD19, FD20, FD21, FD22, FD23, FD24, FD5, FD6, FD7, FD8, FD9: FIDUCIAL1X2, SparkFun-Aesthetics:FIDUCIAL-1X2
- added H10, H11, H12, H13, H14, H15, H16, H17, H18, H19, H20, H21, H22, H23, H24, H5, H6, H7, H8, H9: STAND-OFF, SparkFun-Hardware:STAND-OFF
- added J10, J13, J14, J17, J18, J21, J22, J5, J6, J9: (no value), SparkFun-Connectors:JST04_1MM_RA
- added J11, J12, J15, J16, J19, J20, J23, J24, J7, J8: (no value), SparkFun-Connectors:1X06_NO_SILK
- added JP1, JP13, JP17, JP21, JP9: AUX, SparkFun-Jumpers:SMT-JUMPER_3_2-NC_TRACE_SILK
- added JP10, JP14, JP18, JP22, JP6: I2C PU, SparkFun-Jumpers:SMT-JUMPER_3_2-NC_TRACE_SILK
- added JP11, JP15, JP19, JP23, JP7: LED, SparkFun-Jumpers:SMT-JUMPER_2_NC_TRACE_SILK
- added JP12, JP16, JP20, JP24, JP8: ADR, SparkFun-Jumpers:SMT-JUMPER_2_NO_SILK
- added LOGO10, LOGO12, LOGO4, LOGO6, LOGO8: OSHW-LOGOMINI, SparkFun-Aesthetics:OSHW-LOGO-MINI
- added LOGO11, LOGO3, LOGO5, LOGO7, LOGO9: SFE_LOGO_NAME_FLAME.1_INCH, SparkFun-Aesthetics:SFE_LOGO_NAME_FLAME_.1
- added Q17, Q19, Q21, Q23, Q25, Q27, Q29, Q31, Q33, Q35, Q37, Q39, Q41, Q43, Q45, Q47, Q49, Q51, Q53, Q55, Q57, Q59, Q61, Q63, Q65, Q67, Q69, Q71, Q73, Q75, Q77, Q79, Q81, Q83, Q85, Q87, Q89, Q91, Q93, Q95: DMN2005LP4K-7, new_fets:AP02001
- added Q18, Q20, Q22, Q24, Q26, Q28, Q30, Q32, Q34, Q36, Q38, Q40, Q42, Q44, Q46, Q48, Q50, Q52, Q54, Q56, Q58, Q60, Q62, Q64, Q66, Q68, Q70, Q72, Q74, Q76, Q78, Q80, Q82, Q84, Q86, Q88, Q90, Q92, Q94, Q96: RE1C002UN, new_fets:SOT-416FL
- added R1, R35, R52, R69, R86: 470, SparkFun-Resistors:0603
- added R100, R101, R102, R2, R26, R27, R28, R29, R3, R30, R31, R32, R33, R34, R36, R37, R38, R39, R4, R40, R41, R42, R43, R44, R45, R46, R47, R48, R49, R5, R50, R51, R53, R54, R55, R56, R57, R58, R59, R6, R60, R61, R62, R63, R64, R65, R66, R67, R68, R7, R70, R71, R72, R73, R74, R75, R76, R77, R78, R79, R8, R80, R81, R82, R83, R84, R85, R87, R88, R89, R90, R91, R92, R93, R94, R95, R96, R97, R98, R99: 2.2k, SparkFun-Resistors:0402-TIGHT
- added TP2, TP3, TP4, TP5, TP6: 1.8V, SparkFun-Connectors:PAD.03X.03
- added U$100, U$133, U$142, U$175, U$184, U$217, U$226, U$49, U$58, U$91: (no value), buzzard_labels_2:ADA0
- added U$101, U$132, U$143, U$174, U$185, U$216, U$227, U$48, U$59, U$90: (no value), buzzard_labels_2:ACL1
- added U$102, U$131, U$144, U$173, U$186, U$215, U$228, U$47, U$60, U$89: (no value), buzzard_labels_2:FSNC2
- added U$103, U$130, U$145, U$172, U$187, U$214, U$229, U$46, U$61, U$88: (no value), buzzard_labels_2:INT3
- added U$104, U$126, U$128, U$129, U$146, U$168, U$170, U$171, U$188, U$210, U$212, U$213, U$230, U$252, U$32, U$33, U$62, U$84, U$86, U$87: (no value), buzzard_labels_2:GND4
- added U$105, U$147, U$189, U$231, U$63: (no value), buzzard_labels_2:SPI19
- added U$106, U$148, U$190, U$232, U$64: (no value), buzzard_labels_2:I2C_PU21
- added U$107, U$149, U$191, U$233, U$65: (no value), buzzard_labels_2:AUX_PU24
- added U$108, U$150, U$192, U$234, U$66: (no value), buzzard_labels_2:LED23
- added U$109, U$115, U$151, U$157, U$193, U$199, U$235, U$241, U$67, U$73: (no value), buzzard_labels (1):X0
- added U$110, U$116, U$152, U$158, U$194, U$200, U$236, U$242, U$68, U$74: (no value), buzzard_labels (1):Y1
- added U$111, U$117, U$153, U$159, U$195, U$201, U$237, U$243, U$69, U$75: (no value), buzzard_labels (1):Z2
- added U$112, U$154, U$196, U$238, U$70: (no value), buzzard_labels (1):G5
- added U$113, U$155, U$197, U$239, U$71: (no value), buzzard_labels (1):A4
- added U$114, U$156, U$198, U$240, U$72: (no value), buzzard_labels (1):M3
- added U$118, U$160, U$202, U$244, U$76: (no value), buzzard_labels:QWIIC_9DOF_IMU_0
- added U$119, U$161, U$203, U$245, U$77: (no value), buzzard_labels:CL4
- added U$120, U$162, U$204, U$246, U$78: (no value), buzzard_labels:DA2
- added U$121, U$122, U$139, U$163, U$164, U$181, U$205, U$206, U$223, U$247, U$248, U$55, U$79, U$80, U$97: (no value), buzzard_labels_2:VIN5
- added U$123, U$165, U$207, U$249, U$81: (no value), buzzard_labels_4:PWR0
- added U$124, U$166, U$208, U$250, U$82: (no value), buzzard_labels_4:I#C1
- added U$125, U$167, U$209, U$251, U$83: (no value), buzzard_labels_4:ADR2
- added U$127, U$169, U$211, U$28, U$85: (no value), buzzard_labels:ICM#2094820
- added U$134, U$176, U$218, U$50, U$92: (no value), buzzard_labels_2:MISO13
- added U$135, U$177, U$219, U$51, U$93: (no value), buzzard_labels_2:MOSI14
- added U$136, U$178, U$220, U$52, U$94: (no value), buzzard_labels_2:SCLK15
- added U$137, U$179, U$221, U$53, U$95: (no value), buzzard_labels_2:#CS16
- added U$138, U$180, U$222, U$54, U$96: (no value), buzzard_labels_2:1V8#5V57
- added U$140, U$182, U$224, U$56, U$98: (no value), buzzard_labels_2:NC17
- added U$141, U$183, U$225, U$57, U$99: (no value), buzzard_labels_2:AD012
- added U100, U101, U102, U103, U104, U105, U106, U107, U108, U21, U22, U23, U24, U25, U26, U27, U28, U29, U30, U31, U32, U33, U34, U35, U36, U39, U40, U41, U42, U43, U44, U45, U46, U47, U48, U49, U50, U51, U52, U53, U54, U57, U58, U59, U60, U61, U62, U63, U64, U65, U66, U67, U68, U69, U70, U71, U72, U75, U76, U77, U78, U79, U80, U81, U82, U83, U84, U85, U86, U87, U88, U89, U90, U93, U94, U95, U96, U97, U98, U99: TP, new_fets:MINI_TEST_POINT
- added U19, U37, U55, U73, U91: 1.8V/100mA, SparkFun-IC-Power:SC70
- added U20, U38, U56, U74, U92: 9DoF IMU, SparkFun-Sensors:QFN24-3X3
- moved U$25 1.02 mm to (5.46, 7.62)
Connections:
- net N$2 renamed SCL/SCLK_VIN_JMP
- net N$3 renamed SDA/SDI_VIN_JMP
- net N$4 renamed AUX_CL_VIN_JMP
- net N$5 renamed AUX_DA_VIN_JMP
- new net !CS!_VIN1: J7.6, Q17.D, Q18.3, R3.1, U36.P$1
- new net !CS!_VIN2: J11.6, Q33.D, Q34.3, R37.1, U54.P$1
- new net !CS!_VIN3: J15.6, Q49.D, Q50.3, R54.1, U72.P$1
- new net !CS!_VIN4: J19.6, Q65.D, Q66.3, R71.1, U90.P$1
- new net !CS!_VIN5: J23.6, Q81.D, Q82.3, R88.1, U108.P$1
- new net !CS1: Q17.S, Q18.2, R2.1, U20.22, U35.P$1
- new net !CS2: Q33.S, Q34.2, R36.1, U38.22, U53.P$1
- new net !CS3: Q49.S, Q50.2, R53.1, U56.22, U71.P$1
- new net !CS4: Q65.S, Q66.2, R70.1, U74.22, U89.P$1
- new net !CS5: Q81.S, Q82.2, R87.1, U107.P$1, U92.22
- new net 1.8V1: C6.1, C7.1, D2.A, Q17.G, Q18.1, Q19.G, Q20.1, Q21.G, Q22.1, Q23.G, Q24.1, Q25.G, Q26.1, Q27.G, Q28.1, Q29.G, Q30.1, Q31.G, Q32.1, R2.2, R27.2, R29.2, R31.2, R33.2, R4.2, R6.2, R8.2, TP2.P$1, U19.5, U20.13, U20.8
- new net 1.8V2: C10.1, C11.1, D3.A, Q33.G, Q34.1, Q35.G, Q36.1, Q37.G, Q38.1, Q39.G, Q40.1, Q41.G, Q42.1, Q43.G, Q44.1, Q45.G, Q46.1, Q47.G, Q48.1, R36.2, R38.2, R40.2, R42.2, R44.2, R46.2, R48.2, R50.2, TP3.P$1, U37.5, U38.13, U38.8
- new net 1.8V3: C14.1, C15.1, D4.A, Q49.G, Q50.1, Q51.G, Q52.1, Q53.G, Q54.1, Q55.G, Q56.1, Q57.G, Q58.1, Q59.G, Q60.1, Q61.G, Q62.1, Q63.G, Q64.1, R53.2, R55.2, R57.2, R59.2, R61.2, R63.2, R65.2, R67.2, TP4.P$1, U55.5, U56.13, U56.8
- new net 1.8V4: C18.1, C19.1, D5.A, Q65.G, Q66.1, Q67.G, Q68.1, Q69.G, Q70.1, Q71.G, Q72.1, Q73.G, Q74.1, Q75.G, Q76.1, Q77.G, Q78.1, Q79.G, Q80.1, R70.2, R72.2, R74.2, R76.2, R78.2, R80.2, R82.2, R84.2, TP5.P$1, U73.5, U74.13, U74.8
- new net 1.8V5: C22.1, C23.1, D6.A, Q81.G, Q82.1, Q83.G, Q84.1, Q85.G, Q86.1, Q87.G, Q88.1, Q89.G, Q90.1, Q91.G, Q92.1, Q93.G, Q94.1, Q95.G, Q96.1, R101.2, R87.2, R89.2, R91.2, R93.2, R95.2, R97.2, R99.2, TP6.P$1, U91.5, U92.13, U92.8
- new net AD0/SDO1: Q19.S, Q20.2, R4.1, U20.9, U33.P$1
- new net AD0/SDO2: Q35.S, Q36.2, R38.1, U38.9, U51.P$1
- new net AD0/SDO3: Q51.S, Q52.2, R55.1, U56.9, U69.P$1
- new net AD0/SDO4: Q67.S, Q68.2, R72.1, U74.9, U87.P$1
- new net AD0/SDO5: Q83.S, Q84.2, R89.1, U105.P$1, U92.9
- new net AD0/SDO_VIN1: J7.5, JP8.2, Q19.D, Q20.3, R5.1, U34.P$1
- new net AD0/SDO_VIN2: J11.5, JP12.2, Q35.D, Q36.3, R39.1, U52.P$1
- new net AD0/SDO_VIN3: J15.5, JP16.2, Q51.D, Q52.3, R56.1, U70.P$1
- new net AD0/SDO_VIN4: J19.5, JP20.2, Q67.D, Q68.3, R73.1, U88.P$1
- new net AD0/SDO_VIN5: J23.5, JP24.2, Q83.D, Q84.3, R90.1, U106.P$1
- new net AUX_CL1: Q27.S, Q28.2, R29.1, U20.7, U23.P$1
- new net AUX_CL2: Q43.S, Q44.2, R46.1, U38.7, U41.P$1
- new net AUX_CL3: Q59.S, Q60.2, R63.1, U56.7, U59.P$1
- new net AUX_CL4: Q75.S, Q76.2, R80.1, U74.7, U77.P$1
- new net AUX_CL5: Q91.S, Q92.2, R97.1, U92.7, U95.P$1
- new net AUX_CL_VIN1: J8.5, Q27.D, Q28.3, R30.1, U24.P$1
- new net AUX_CL_VIN2: J12.5, Q43.D, Q44.3, R47.1, U42.P$1
- new net AUX_CL_VIN3: J16.5, Q59.D, Q60.3, R64.1, U60.P$1
- new net AUX_CL_VIN4: J20.5, Q75.D, Q76.3, R81.1, U78.P$1
- new net AUX_CL_VIN5: J24.5, Q91.D, Q92.3, R98.1, U96.P$1
- new net AUX_CL_VIN_JMP1: JP1.1, R30.2
- new net AUX_CL_VIN_JMP2: JP9.1, R47.2
- new net AUX_CL_VIN_JMP3: JP13.1, R64.2
- new net AUX_CL_VIN_JMP4: JP17.1, R81.2
- new net AUX_CL_VIN_JMP5: JP21.1, R98.2
- new net AUX_DA1: Q25.S, Q26.2, R27.1, U20.21, U21.P$1
- new net AUX_DA2: Q41.S, Q42.2, R44.1, U38.21, U39.P$1
- new net AUX_DA3: Q57.S, Q58.2, R61.1, U56.21, U57.P$1
- new net AUX_DA4: Q73.S, Q74.2, R78.1, U74.21, U75.P$1
- new net AUX_DA5: Q89.S, Q90.2, R95.1, U92.21, U93.P$1
- new net AUX_DA_VIN1: J8.4, Q25.D, Q26.3, R28.1, U22.P$1
- new net AUX_DA_VIN2: J12.4, Q41.D, Q42.3, R45.1, U40.P$1
- new net AUX_DA_VIN3: J16.4, Q57.D, Q58.3, R62.1, U58.P$1
- new net AUX_DA_VIN4: J20.4, Q73.D, Q74.3, R79.1, U76.P$1
- new net AUX_DA_VIN5: J24.4, Q89.D, Q90.3, R96.1, U94.P$1
- new net AUX_DA_VIN_JMP1: JP1.3, R28.2
- new net AUX_DA_VIN_JMP2: JP9.3, R45.2
- new net AUX_DA_VIN_JMP3: JP13.3, R62.2
- new net AUX_DA_VIN_JMP4: JP17.3, R79.2
- new net AUX_DA_VIN_JMP5: JP21.3, R96.2
- new net FSYNC1: Q29.S, Q30.2, R31.1, U20.11, U26.P$1
- new net FSYNC2: Q45.S, Q46.2, R48.1, U38.11, U44.P$1
- new net FSYNC3: Q61.S, Q62.2, R65.1, U56.11, U62.P$1
- new net FSYNC4: Q77.S, Q78.2, R82.1, U74.11, U80.P$1
- new net FSYNC5: Q93.S, Q94.2, R99.1, U92.11, U98.P$1
- new net FSYNC_VIN1: J8.3, Q29.D, Q30.3, R32.1, U25.P$1
- new net FSYNC_VIN2: J12.3, Q45.D, Q46.3, R49.1, U43.P$1
- new net FSYNC_VIN3: J16.3, Q61.D, Q62.3, R66.1, U61.P$1
- new net FSYNC_VIN4: J20.3, Q77.D, Q78.3, R83.1, U79.P$1
- new net FSYNC_VIN5: J24.3, Q93.D, Q94.3, R100.1, U97.P$1
- new net GND1: C5.2, C6.2, C7.2, C8.2, J5.1, J6.1, J7.1, J8.1, JP7.1, JP8.1, U19.2, U20.18, U20.20
- new net GND2: C10.2, C11.2, C12.2, C9.2, J10.1, J11.1, J12.1, J9.1, JP11.1, JP12.1, U37.2, U38.18, U38.20
- new net GND3: C13.2, C14.2, C15.2, C16.2, J13.1, J14.1, J15.1, J16.1, JP15.1, JP16.1, U55.2, U56.18, U56.20
- new net GND4: C17.2, C18.2, C19.2, C20.2, J17.1, J18.1, J19.1, J20.1, JP19.1, JP20.1, U73.2, U74.18, U74.20
- new net GND5: C21.2, C22.2, C23.2, C24.2, J21.1, J22.1, J23.1, J24.1, JP23.1, JP24.1, U91.2, U92.18, U92.20
- new net INT1: Q31.S, Q32.2, R33.1, U20.12, U27.P$1
- new net INT2: Q47.S, Q48.2, R50.1, U38.12, U45.P$1
- new net INT3: Q63.S, Q64.2, R67.1, U56.12, U63.P$1
- new net INT4: Q79.S, Q80.2, R84.1, U74.12, U81.P$1
- new net INT5: Q95.S, Q96.2, R101.1, U92.12, U99.P$1
- new net INT_VIN1: J8.2, Q31.D, Q32.3, R34.1, U28.P$1
- new net INT_VIN2: J12.2, Q47.D, Q48.3, R51.1, U46.P$1
- new net INT_VIN3: J16.2, Q63.D, Q64.3, R68.1, U64.P$1
- new net INT_VIN4: J20.2, Q79.D, Q80.3, R85.1, U82.P$1
- new net INT_VIN5: J24.2, Q95.D, Q96.3, R102.1, U100.P$1
- new net N$12: C13.1, U56.10
- new net N$13: D4.C, R52.2
- new net N$14: JP15.2, R52.1
- new net N$16: C17.1, U74.10
- new net N$17: D5.C, R69.2
- new net N$18: JP19.2, R69.1
- new net N$2: C5.1, U20.10
- new net N$20: C21.1, U92.10
- new net N$21: D6.C, R86.2
- new net N$22: JP23.2, R86.1
- new net N$3: D2.C, R1.2
- new net N$4: JP7.2, R1.1
- new net N$6: C9.1, U38.10
- new net N$7: D3.C, R35.2
- new net N$8: JP11.2, R35.1
- new net SCL/SCLK1: Q21.S, Q22.2, R6.1, U20.23, U31.P$1
- new net SCL/SCLK2: Q37.S, Q38.2, R40.1, U38.23, U49.P$1
- new net SCL/SCLK3: Q53.S, Q54.2, R57.1, U56.23, U67.P$1
- new net SCL/SCLK4: Q69.S, Q70.2, R74.1, U74.23, U85.P$1
- new net SCL/SCLK5: Q85.S, Q86.2, R91.1, U103.P$1, U92.23
- new net SCL/SCLK_VIN1: J5.4, J6.4, J7.4, Q21.D, Q22.3, R7.1, U32.P$1
- new net SCL/SCLK_VIN2: J10.4, J11.4, J9.4, Q37.D, Q38.3, R41.1, U50.P$1
- new net SCL/SCLK_VIN3: J13.4, J14.4, J15.4, Q53.D, Q54.3, R58.1, U68.P$1
- new net SCL/SCLK_VIN4: J17.4, J18.4, J19.4, Q69.D, Q70.3, R75.1, U86.P$1
- new net SCL/SCLK_VIN5: J21.4, J22.4, J23.4, Q85.D, Q86.3, R92.1, U104.P$1
- new net SCL/SCLK_VIN_JMP1: JP6.3, R7.2
- new net SCL/SCLK_VIN_JMP2: JP10.3, R41.2
- new net SCL/SCLK_VIN_JMP3: JP14.3, R58.2
- new net SCL/SCLK_VIN_JMP4: JP18.3, R75.2
- new net SCL/SCLK_VIN_JMP5: JP22.3, R92.2
- new net SDA/SDI1: Q23.S, Q24.2, R8.1, U20.24, U29.P$1
- new net SDA/SDI2: Q39.S, Q40.2, R42.1, U38.24, U47.P$1
- new net SDA/SDI3: Q55.S, Q56.2, R59.1, U56.24, U65.P$1
- new net SDA/SDI4: Q71.S, Q72.2, R76.1, U74.24, U83.P$1
- new net SDA/SDI5: Q87.S, Q88.2, R93.1, U101.P$1, U92.24
- new net SDA/SDI_VIN1: J5.3, J6.3, J7.3, Q23.D, Q24.3, R26.1, U30.P$1
- new net SDA/SDI_VIN2: J10.3, J11.3, J9.3, Q39.D, Q40.3, R43.1, U48.P$1
- new net SDA/SDI_VIN3: J13.3, J14.3, J15.3, Q55.D, Q56.3, R60.1, U66.P$1
- new net SDA/SDI_VIN4: J17.3, J18.3, J19.3, Q71.D, Q72.3, R77.1, U84.P$1
- new net SDA/SDI_VIN5: J21.3, J22.3, J23.3, Q87.D, Q88.3, R94.1, U102.P$1
- new net SDA/SDI_VIN_JMP1: JP6.1, R26.2
- new net SDA/SDI_VIN_JMP2: JP10.1, R43.2
- new net SDA/SDI_VIN_JMP3: JP14.1, R60.2
- new net SDA/SDI_VIN_JMP4: JP18.1, R77.2
- new net SDA/SDI_VIN_JMP5: JP22.1, R94.2
- new net VIN1: C8.1, J5.2, J6.2, J7.2, J8.6, JP1.2, JP6.2, R3.2, R32.2, R34.2, R5.2, U19.1, U19.3
- new net VIN2: C12.1, J10.2, J11.2, J12.6, J9.2, JP10.2, JP9.2, R37.2, R39.2, R49.2, R51.2, U37.1, U37.3
- new net VIN3: C16.1, J13.2, J14.2, J15.2, J16.6, JP13.2, JP14.2, R54.2, R56.2, R66.2, R68.2, U55.1, U55.3
- new net VIN4: C20.1, J17.2, J18.2, J19.2, J20.6, JP17.2, JP18.2, R71.2, R73.2, R83.2, R85.2, U73.1, U73.3
- new net VIN5: C24.1, J21.2, J22.2, J23.2, J24.6, JP21.2, JP22.2, R100.2, R102.2, R88.2, R90.2, U91.1, U91.3
Routing:
- net 1.8V2: track 0.00 -> 100.8 mm, vias 0 -> 13
- net 1.8V5: track 0.00 -> 100.8 mm, vias 0 -> 13
- net 1.8V3: track 0.00 -> 100.8 mm, vias 0 -> 13
- net 1.8V1: track 0.00 -> 100.8 mm, vias 0 -> 13
- net 1.8V4: track 0.00 -> 100.8 mm, vias 0 -> 13
- net VIN5: track 0.00 -> 88.5 mm, vias 0 -> 7
- net VIN3: track 0.00 -> 88.5 mm, vias 0 -> 7
- net VIN4: track 0.00 -> 88.5 mm, vias 0 -> 7
- net VIN2: track 0.00 -> 88.5 mm, vias 0 -> 7
- net VIN1: track 0.00 -> 88.5 mm, vias 0 -> 7
- net SDA/SDI_VIN3: track 0.00 -> 48.1 mm, vias 0 -> 2
- net SDA/SDI_VIN2: track 0.00 -> 48.1 mm, vias 0 -> 2
- net SDA/SDI_VIN4: track 0.00 -> 48.1 mm, vias 0 -> 2
- net SDA/SDI_VIN5: track 0.00 -> 48.1 mm, vias 0 -> 2
- net SDA/SDI_VIN1: track 0.00 -> 48.1 mm, vias 0 -> 2
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- added copper zone on layer 1, net GND1
- added copper zone on layer 16, net GND1
- added copper zone on layer 1, net GND2
- added copper zone on layer 16, net GND2
- added copper zone on layer 1, net GND3
- added copper zone on layer 16, net GND3
- added copper zone on layer 1, net GND4
- added copper zone on layer 16, net GND4
- added copper zone on layer 1, net GND5
- added copper zone on layer 16, net GND5
Other:
- board size 31.8 x 25.4 mm -> 84.1 x 97.3 mm
- board text added: "v-score"
- board text removed: "Owen Lyke"
